File: mcu/mcu.kicad_sch (KiCad schematic)
At the start: 13 parts, among them J1 SWD connector, U1 STM32F411CEUx, Y1 25MHz 9pF, Y2 32.768kHz 6pF

Commit message: Blinky.
Parts:
- removed C6, C7, C8: 100nF, symbol Device:C
- added D?: SW_LED, symbol Device:LED
- added SW?: RST, symbol Switch:SW_SPST
- added SW?: SW_KEY, symbol Switch:SW_SPST
Connections:
- net GND: now also U1.44 (BOOT0), SW?.2 (B), SW?.2 (B)
- net SWDIO: now also U1.34 (PA13); no longer U1.38 (PA15)
- net VDD: now also D?.2 (A)
- net at U1.10 (PA0): now also SW?.1 (A)
- net sd_cs: now reaches U1.14 (PA4)
- net can1_int: now reaches U1.18 (PB0)
- net can2_int: now reaches U1.19 (PB1)
- net at U1.2 (PC13): now also D?.1 (K)
- net can1_cs: now reaches U1.46 (PB9)
- net at U1.7 (NRST): now also SW?.1 (A)
- new net can2_cs: U1.38 (PA15)
